Commit message: 重组工作空间目录：移入 bbot_demo_roscontrol 与 a3_robot_descriptions，新增 robot_moveit2
- bbot_demo、ros_team_workspace 移至 bbot_demo_roscontrol/ 下
- robot_descriptions 移至 a3_robot_descriptions/src/ 下
- 新增 robot_moveit2 工作空间及测试用 urdf 文件
- 修改 arm.xacro

Co-Authored-By: Claude Code <noreply@anthropic.com>

File: ros2-moveit2-arm-control-tutorial-main/ros2_ws/src/my_robot_description/urdf/test_arm.xacro (robot description, xacro)
@@ -1,5 +1,5 @@
 <?xml version="1.0"?>
 <robot xmlns:xacro="http://www.ros.org/wiki/xacro">
-    <!-- base_link: box size 0.4 0.4 0.1 -->
+     <!-- base_link: box size 0.4 0.4 0.1 -->
     <link name="base_link">
         <visual>
@@ -10,14 +10,5 @@
             <material name="grey"/>
         </visual>
-        <collision>
-            <geometry>
-                <box size="0.4 0.4 0.1"/>
-            </geometry>
-            <origin xyz="0 0 0.05" rpy="0 0 0"/>
-        </collision>
     </link>
-      <gazebo reference="base_link">
-      <material>Gazebo/Orange</material>
-    </gazebo>
     <!-- shoulder_link: cylinder length 0.5 radius 0.1 -->
     <link name="shoulder_link">
@@ -29,14 +20,5 @@
             <material name="blue"/>
         </visual>
-        <collision>
-            <geometry>
-                <box size="0.2 0.2 0.5"/>
-            </geometry>
-            <origin xyz="0 0 0.25" rpy="0 0 0"/>
-        </collision>
     </link>
-     <gazebo reference="shoulder_link">
-        <material>Gazebo/Black</material>
-    </gazebo>
     <!-- arm_link: cylinder length 0.6 radius 0.05 -->
     <link name="arm_link">
@@ -49,14 +31,5 @@
             <material name="grey"/>
         </visual>
-        <collision>
-            <geometry>
-                <box size="0.1 0.1 0.6"/>
-            </geometry>
-            <origin xyz="0 0 0.3" rpy="0 0 0"/>
-        </collision>
     </link>
-      <gazebo reference="arm_link">
-      <material>Gazebo/Gray</material>
-    </gazebo>
     <!-- elbow_link: cylinder length 0.1 radius 0.05 -->
     <link name="elbow_link">
@@ -68,14 +41,5 @@
             <material name="blue"/>
         </visual>
-        <collision>
-            <geometry>
-                <box size="0.1 0.1 0.1"/>
-            </geometry>
-            <origin xyz="0 0 0.05" rpy="0 0 0"/>
-        </collision>
     </link>
-       <gazebo reference="elbow_link">
-      <material>Gazebo/White</material>
-    </gazebo>
     <!-- forearm_link: cylinder length 0.5 radius 0.05 -->
     <link name="forearm_link">
@@ -88,14 +52,5 @@
             <material name="grey"/>
         </visual>
-        <collision>
-            <geometry>
-                <box size="0.1 0.1 0.5"/>
-            </geometry>
-            <origin xyz="0 0 0.25" rpy="0 0 0"/>
-        </collision>
     </link>
-      <gazebo reference="forearm_link">
-      <material>Gazebo/Blue</material>
-    </gazebo>
     <!-- wrist_link: box size 0.1 0.1 0.05 -->
     <link name="wrist_link">
@@ -107,14 +62,5 @@
             <material name="blue"/>
         </visual>
-        <collision>
-            <geometry>
-                <box size="0.1 0.1 0.05"/>
-            </geometry>
-            <origin xyz="0 0 0.025" rpy="0 0 0"/>
-        </collision>
     </link>
-    <gazebo reference="wrist_link">
-      <material>Gazebo/Black</material>
-    </gazebo>
     <!-- hand_link: box size 0.1 0.1 0.02 -->
     <link name="hand_link">
@@ -126,14 +72,5 @@
             <material name="grey"/>
         </visual>
-        <collision>
-            <geometry>
-                <box size="0.1 0.1 0.02"/>
-            </geometry>
-            <origin xyz="0 0 0.01" rpy="0 0 0"/>
-        </collision>
     </link>
-    <gazebo reference="hand_link">
-      <material>Gazebo/White</material>
-    </gazebo>
     <!-- tool_link: no visual -->
     <link name="tool_link"/>
